File: Z50-GDP.kicad_sch (KiCad schematic)
At the start: 59 parts, among them J1 Z50Bus, J2 Conn_01x09, SW0 SW_Push, SW1 SW_Push, SW2 SW_Push, SW3 SW_Push, SW4 SW_Push, SW5 SW_Push, SW6 SW_Push, SW7 SW_Push, SW8 SW_DIP_x08, SW9 SW_DIP_x08, U1 74LS688, U10 74LS299, U11 74HCT273, U2 74LS273, U3 74LS245, U4 74LS32, U5 EF9366, U6 74LS166, U7 74LS374, U8 74LS163, U9 AS6C1008-55PCN

Commit message: Schematic basically ready
Parts:
- removed C1: 100n, Capacitors_THT:C_Disc_D4.7mm_W2.5mm_P5.00mm, symbol Device:C
- removed D0, D1, D2, D3, D4, D5, D6, D7: LED, LEDs:LED_D5.0mm, symbol Device:LED
- removed J2: Conn_01x09, Pin_Headers:Pin_Header_Straight_1x09_Pitch2.54mm, symbol Connector_Generic:Conn_01x09
- removed R0, R1, R2, R24, R3, R4, R5, R6, R7: 4k7, Resistors_THT:R_Axial_DIN0207_L6.3mm_D2.5mm_P10.16mm_Horizontal, symbol Device:R
- removed R10, R11, R12, R13, R14, R15, R8, R9: 2k, Resistors_THT:R_Axial_DIN0207_L6.3mm_D2.5mm_P10.16mm_Horizontal, symbol Device:R
- removed R16, R17, R18, R19, R20, R21, R22, R23: 330, Resistors_THT:R_Axial_DIN0207_L6.3mm_D2.5mm_P10.16mm_Horizontal, symbol Device:R
- removed SW0, SW1, SW2, SW3, SW4, SW5, SW6, SW7: SW_Push, Buttons_Switches_THT:SW_PUSH_6mm, symbol Switch:SW_Push
- removed SW8, SW9: SW_DIP_x08, Buttons_Switches_THT:SW_DIP_x8_W7.62mm_Piano, symbol Switch:SW_DIP_x08
- removed U1: 74LS688, Housings_DIP:DIP-20_W7.62mm_Socket_LongPads, symbol 74xx:74LS688
- removed U2: 74LS273, Housings_DIP:DIP-20_W7.62mm_Socket_LongPads, symbol 74xx:74LS273
- removed U3: 74LS245, Housings_DIP:DIP-20_W7.62mm_Socket_LongPads, symbol 74xx:74LS245
- removed U4 (x3): 74LS32, Housings_DIP:DIP-14_W7.62mm_Socket_LongPads, symbol 74xx:74LS32
- removed U9: AS6C1008-55PCN, AS6C1008-55PCN:DIP1524W45P254L4191H419Q32, symbol AS6C1008-55PCN:AS6C1008-55PCN
- added IC1: UM61512A, symbol memory-umc:UM61512A
- added J3: Conn_02x06_Odd_Even, Connector_PinHeader_2.54mm:PinHeader_2x06_P2.54mm_Vertical, symbol Connector_Generic:Conn_02x06_Odd_Even
- added J4: Conn_01x06, Connector_PinHeader_2.54mm:PinHeader_1x06_P2.54mm_Vertical, symbol Connector_Generic:Conn_01x06
- added J5: DE9_Plug_MountingHoles, Connector_Dsub:DSUB-9_Male_Horizontal_P2.77x2.84mm_EdgePinOffset4.94mm_Housed_MountingHolesOffset7.48mm, symbol Connector:DE9_Plug_MountingHoles
- added J6: Conn_Coaxial, Connector_Coaxial:BNC_Amphenol_B6252HB-NPP3G-50_Horizontal, symbol Connector:Conn_Coaxial
- added J7: Conn_02x04_Odd_Even, Connector_PinHeader_2.54mm:PinHeader_2x04_P2.54mm_Vertical, symbol Connector_Generic:Conn_02x04_Odd_Even
- added Q1: BC107, Package_TO_SOT_THT:TO-18-3, symbol Transistor_BJT:BC107
- added R25, R34, R37, R38, R39, R40: 1k, symbol Device:R
- added R26: 75, symbol Device:R
- added R27: 150, symbol Device:R
- added R28, R29, R31, R32, R33, R35, R36: 470, symbol Device:R
- added R30: 220, symbol Device:R
- added U12, U16: 74LS00, symbol 74xx:74LS00
- added U13: 74LS05, symbol 74xx:74LS05
- added U14, U15, U17: 74LS32, symbol 74xx:74LS32
- added U18: 74LS85, symbol 74xx:74LS85
- added U19, U20, U9: 74LS04, symbol 74xx:74LS04
- added U21: 74LS08, symbol 74xx:74LS08
- added X1: 14 MHz, Oscillator:Oscillator_DIP-8, symbol Oscillator:CXO_DIP8
Connections:
- net A0: now also U5.9 (A0)
- net A1: now also U5.10 (A1), U21.5
- net A2: now also U5.11 (A2), U21.2
- net A3: now also U5.12 (A3), U21.1
- net A4: now also U18.10 (A0)
- net A5: now also U18.12 (A1)
- net A6: now also U18.13 (A2)
- net A7: now also U18.15 (A3)
- net D0: now also U5.33 (D0), U7.2 (O0)
- net D1: now also U5.32 (D1), U7.5 (O1)
- net D2: now also U5.31 (D2), U7.6 (O2)
- net D3: now also U5.30 (D3), U7.9 (O3)
- net D4: now also U5.29 (D4), U7.12 (O4)
- net D5: now also U5.28 (D5), U7.15 (O5)
- net D6: now also U5.27 (D6), U7.16 (O6)
- net D7: now also U5.26 (D7), U7.19 (O7)
- net GND: now also U10.1 (S0), U10.10 (GND), U11.10 (GND), U11.18 (D7), U5.23 (WO), U6.1 (Ds), U6.6 (CE), U6.8 (GND), U7.10 (GND), U8.3 (D0), U8.4 (D1), U8.5 (D2), U8.8 (GND), IC1.16 (GND), IC1.3 (A14), IC1.31 (A15), J4.5 (Pin_5), J4.6 (Pin_6), J5.1, J5.2, J6.2 (Ext), J7.1 (Pin_1), J7.3 (Pin_3), J7.5 (Pin_5), J7.7 (Pin_7), R25.2, R28.2, U18.2 (Ia<b), U18.4 (Ia>b), U18.8 (GND), X1.4 (GND)
- net ~{IOREQ}: now also U20.1
- net ~{WR}: now also U5.18 (R/~{W}), U21.12
- net ~{INT}: now reaches J1.24 (Pin_24)
- net ~{INT}: now also U5.13 (~{IRQ}), R40.2
- net at U11.11 (Cp): now also U10.12 (Cp), U5.1 (CK), U8.12 (Q2), U12.2
- net at U11.12 (Q4): now also IC1.8 (A4)
- net at U11.15 (Q5): now also IC1.7 (A5)
- net at U11.16 (Q6): now also IC1.6 (A6)
- net at U11.2 (Q0): now also IC1.12 (A0)
- net +5V: now reaches U11.20 (VCC)
- net +5V: now also U10.11 (Ds0), U10.19 (S1), U10.20 (VCC), U5.21 (LPCK), U5.8 (FMAT), U6.16 (VCC), U7.20 (VCC), U8.1 (~{MR}), U8.10 (CET), U8.16 (VCC), U8.6 (D3), U8.7 (CEP), IC1.30 (CE2), IC1.32 (VCC), Q1.3 (C), R29.1, R30.1, R31.1, R32.1, R33.1, R34.1, R35.1, R36.1, R37.1, R38.1, R39.1, R40.1, U18.16 (VCC), X1.1 (EN), X1.8 (Vcc)
- net at U11.5 (Q1): now also IC1.11 (A1)
- net at U11.6 (Q2): now also IC1.10 (A2)
- net at U11.9 (Q3): now also IC1.9 (A3)
- net at U6.10 (E): now also U10.5 (IO4), U7.13 (D4), IC1.18 (D4)
- net at U6.11 (F): now also U10.15 (IO5), U7.14 (D5), IC1.19 (D5)
- net at U6.12 (G): now also U10.4 (IO6), U7.17 (D6), IC1.20 (D6)
- net at U6.13 (Qh): now also J3.11 (Pin_11), U13.5, U17.1
- net at U6.14 (H): now also U10.16 (IO7), U7.18 (D7), IC1.21 (D7)
- net at U6.15 (PE): now also U14.3
- net at U6.2 (A): now also U10.7 (IO0), U7.3 (D0), IC1.13 (D0)
- net at U6.3 (B): now also U10.13 (IO1), U7.4 (D1), IC1.14 (D1)
- net at U6.4 (C): now also U10.6 (IO2), U7.7 (D2), IC1.15 (D2)
- net at U6.5 (D): now also U10.14 (IO3), U7.8 (D3), IC1.17 (D3)
- net 14M: now reaches U6.7 (Clk)
- net 14M: now also U8.2 (CP), U17.2, X1.5 (OUT)
- net at U6.9 (Clr): now also U5.24 (~{WHITE})
- net at U7.1 (OE): now also U21.11
- net at U7.11 (Cp): now also U15.3
- net at U10.18 (Ds7): now also U5.15 (DIN)
- net at U10.2 (OE1): now also U10.3 (OE2), U12.4, U12.5, U16.3
- net at U10.9 (Mr): now also IC1.24 (OE), U12.6
- net at U8.13 (Q1): now also U12.1
- net at U8.15 (TC): now also U9.1
- net at U8.9 (~{PE}): now also U14.2, U15.2, U9.2
- net at U5.14 (~{DW}): now also IC1.29 (WR)
- net at U5.16 (VB): now also J3.7 (Pin_7), R35.2, U13.3
- net at U5.17 (~{E}): now also U19.2
- net at U5.19 (~{MFREE}): now also U15.1, U16.2
- net at U5.22 (~{ALL}): now also U16.1
- net at U5.25 (BLK): now also U14.1
- net at U5.34 (SYNC): now also U13.11, U13.13
- new net: R27.2, R28.1, U13.8
- new net: U13.9, U17.3
- new net: J3.9 (Pin_9), R32.2, U13.6
- new net: J3.3 (Pin_3), R36.2, U13.1, U13.12
- new net: U18.3 (Ia=b), U20.2
- new net: Q1.2 (B), R27.1, R29.2, U13.10
- new net: J5.6, R30.2
- new net: U21.10, U21.6
- new net: U21.13, U21.8
- new net: U18.6 (Oa=b), U19.1, U21.9
- new net: J7.2 (Pin_2), R38.2, U18.1 (B3)
- new net: J7.4 (Pin_4), R37.2, U18.14 (B2)
- new net: J7.6 (Pin_6), R34.2, U18.11 (B1)
- new net: J7.8 (Pin_8), R39.2, U18.9 (B0)
- new net: Q1.1 (E), R25.1, R26.1
- new net: U21.3, U21.4
- new net: J3.1 (Pin_1), R31.2, U13.2
- new net: J3.5 (Pin_5), R33.2, U13.4
- new net BAS: J4.1 (Pin_1), J6.1 (In), R26.2
- new net HS: J3.2 (Pin_2), J3.4 (Pin_4), J4.2 (Pin_2), J5.8
- new net VI: J3.10 (Pin_10), J3.12 (Pin_12), J3.6 (Pin_6), J3.8 (Pin_8), J4.3 (Pin_3), J4.4 (Pin_4), J5.7, J5.9
- new net ~{CAS}: IC1.22 (CE1), U12.3
- no-connect marks 26 -> 36
Other:
- moved on the sheet: J1, U10, U11, U5A, U6, U7, U8

Commit message: Schematic annotated
Parts:
- removed unit 4 of U21
- added C1, C10, C11, C12, C13, C2, C3, C4, C5, C6, C7, C8, C9: 100n, Capacitor_THT:C_Rect_L4.0mm_W2.5mm_P2.50mm, symbol Device:C
- added unit 4 of U2
- added unit 4 of U5
- added unit 7 of U5
- added unit 6 of U5
- added unit 5 of U5
- added unit 5 of U6
- added unit 4 of U6
- added unit 4 of U8
- added unit 5 of U8
- IC1: footprint (none) -> Package_DIP:DIP-32_W7.62mm
- J2: renamed from J1; footprint Pin_Headers:Pin_Header_Straight_2x25_Pitch2.54mm -> Connector_PinHeader_2.54mm:PinHeader_2x25_P2.54mm_Horizontal
- R1: renamed from R39; footprint (none) -> Resistor_THT:R_Axial_DIN0207_L6.3mm_D2.5mm_P10.16mm_Horizontal
- R10: renamed from R28; footprint (none) -> Resistor_THT:R_Axial_DIN0207_L6.3mm_D2.5mm_P10.16mm_Horizontal
- R11: renamed from R33; footprint (none) -> Resistor_THT:R_Axial_DIN0207_L6.3mm_D2.5mm_P10.16mm_Horizontal
- R12: renamed from R32; footprint (none) -> Resistor_THT:R_Axial_DIN0207_L6.3mm_D2.5mm_P10.16mm_Horizontal
- R13: renamed from R31; footprint (none) -> Resistor_THT:R_Axial_DIN0207_L6.3mm_D2.5mm_P10.16mm_Horizontal
- R14: renamed from R25; footprint (none) -> Resistor_THT:R_Axial_DIN0207_L6.3mm_D2.5mm_P10.16mm_Horizontal
- R15: renamed from R30; footprint (none) -> Resistor_THT:R_Axial_DIN0207_L6.3mm_D2.5mm_P10.16mm_Horizontal
- R16: renamed from R26; footprint (none) -> Resistor_THT:R_Axial_DIN0207_L6.3mm_D2.5mm_P10.16mm_Horizontal
- R2: renamed from R34; footprint (none) -> Resistor_THT:R_Axial_DIN0207_L6.3mm_D2.5mm_P10.16mm_Horizontal
- R3: renamed from R37; footprint (none) -> Resistor_THT:R_Axial_DIN0207_L6.3mm_D2.5mm_P10.16mm_Horizontal
- R4: renamed from R38; footprint (none) -> Resistor_THT:R_Axial_DIN0207_L6.3mm_D2.5mm_P10.16mm_Horizontal
- R5: renamed from R40; footprint (none) -> Resistor_THT:R_Axial_DIN0207_L6.3mm_D2.5mm_P10.16mm_Horizontal
- R6: renamed from R35; footprint (none) -> Resistor_THT:R_Axial_DIN0207_L6.3mm_D2.5mm_P10.16mm_Horizontal
- R7: renamed from R36; footprint (none) -> Resistor_THT:R_Axial_DIN0207_L6.3mm_D2.5mm_P10.16mm_Horizontal
- R8: renamed from R29; footprint (none) -> Resistor_THT:R_Axial_DIN0207_L6.3mm_D2.5mm_P10.16mm_Horizontal
- R9: renamed from R27; footprint (none) -> Resistor_THT:R_Axial_DIN0207_L6.3mm_D2.5mm_P10.16mm_Horizontal
- U1: renamed from U5; footprint (none) -> Package_DIP:DIP-40_W25.4mm
- U10: footprint (none) -> Package_DIP:DIP-20_W7.62mm
- U11: renamed from U7; footprint (none) -> Package_DIP:DIP-20_W7.62mm
- U12: renamed from U6; footprint (none) -> Package_DIP:DIP-16_W7.62mm
- U2: renamed from U21; footprint (none) -> Package_DIP:DIP-14_W7.62mm
- U3: renamed from U13; footprint (none) -> Package_DIP:DIP-14_W7.62mm
- U4: renamed from U18; footprint (none) -> Package_DIP:DIP-16_W7.62mm
- U5: renamed from U20; footprint (none) -> Package_DIP:DIP-14_W7.62mm
- U5: renamed from U9; footprint (none) -> Package_DIP:DIP-14_W7.62mm
- U5: renamed from U19; footprint (none) -> Package_DIP:DIP-14_W7.62mm
- U6: renamed from U12; footprint (none) -> Package_DIP:DIP-14_W7.62mm
- U6: renamed from U16; footprint (none) -> Package_DIP:DIP-14_W7.62mm
- U7: renamed from U8; footprint (none) -> Package_DIP:DIP-16_W7.62mm
- U8: renamed from U15; footprint (none) -> Package_DIP:DIP-14_W7.62mm
- U8: renamed from U14; footprint (none) -> Package_DIP:DIP-14_W7.62mm
- U8: renamed from U17; footprint (none) -> Package_DIP:DIP-14_W7.62mm
- U9: renamed from U11; footprint (none) -> Package_DIP:DIP-20_W7.62mm
- renumbered J7 to J1, J6 to J4, J4 to J5, J5 to J6
Connections:
- net VCC is gone; now on net +5V: J2.19 (Pin_19), J2.20 (Pin_20)
- net +5V: now also U1.40 (VCC), U2.14 (VCC), U3.14 (VCC), U9.1 (~{Mr}), C1.1, C10.1, C11.1, C12.1, C13.1, C2.1, C3.1, C4.1, C5.1, C6.1, C7.1, C8.1, C9.1, U5.14 (VCC), U6.14 (VCC), U8.14 (VCC)
- net 14M: now also U8.10; no longer U8.2
- net GND: now also J6.0 (PAD), U1.20 (GND), U2.7 (GND), U3.7 (GND), C1.2, C10.2, C11.2, C12.2, C13.2, C2.2, C3.2, C4.2, C5.2, C6.2, C7.2, C8.2, C9.2, U2.12, U2.13, U5.11, U5.13, U5.7 (GND), U5.9, U6.7 (GND), U8.12, U8.13, U8.7 (GND)
- net VI: no longer J3.6 (Pin_6), J3.8 (Pin_8), J5.3 (Pin_3), J6.9
- net ~{CAS}: now also U6.8; no longer U6.3
- net ~{WR}: now also U6.12
- net at U3.9: now also U8.8; no longer U8.3
- net at U1.1 (CK), U10.12 (Cp), U7.12 (Q2)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: now also U6.10; no longer U6.2
- net DAD2: now reaches U1.38 (DAD2), U9.13 (D4)
- net DAD2: now also IC1.25 (A11)
- net DAD1: now reaches U1.39 (DAD1), U9.14 (D5)
- net DAD1: now also IC1.4 (A12)
- net DAD0: now reaches U1.37 (DAD0), U9.17 (D6)
- net DAD0: now also IC1.28 (A13)
- net DAD6: now reaches U1.5 (DAD6), U9.3 (D0)
- net DAD6: now also IC1.5 (A7)
- net DAD5: now reaches U1.2 (DAD5), U9.4 (D1)
- net DAD5: now also IC1.27 (A8)
- net DAD4: now reaches U1.3 (DAD4), U9.7 (D2)
- net DAD4: now also IC1.26 (A9)
- net DAD3: now reaches U1.4 (DAD3), U9.8 (D3)
- net DAD3: now also IC1.23 (A10)
- net at J3.11 (Pin_11), U12.13 (Qh), U3.5: now also U8.9; no longer U8.1
- net at U7.15 (TC): now also U5.5; no longer U5.1
- net at U7.9 (~{PE}), U8.2: now also U5.6, U8.5; no longer U5.2, U8.2
- net at U1.19 (~{MFREE}), U6.2: now also U8.4; no longer U8.1
- net at U11.11 (Cp): now also U8.6; no longer U8.3
- net at U2.8: now also U6.13
- net at U2.9, U4.6 (Oa=b): now also U5.3; no longer U5.1
- net at U11.1 (OE): now also U6.11
- net at U7.13 (Q1): now also U6.9; no longer U6.1
- net at U1.17 (~{E}): now also U5.4; no longer U5.2
- net ~{RD}: no longer names the net of J2.28 (Pin_28)
- net ~{RESET}: no longer names the net of J2.22 (Pin_22)
- new net VS: J3.6 (Pin_6), J3.8 (Pin_8), J5.3 (Pin_3), J6.9
- no-connect marks 36 -> 43
Other:
- moved on the sheet: U2E, U3G

Commit message: Routing completed
Parts:
- removed J1: Conn_02x04_Odd_Even, Connector_PinHeader_2.54mm:PinHeader_2x04_P2.54mm_Vertical, symbol Connector_Generic:Conn_02x04_Odd_Even
- removed R1, R2, R3, R4, R5: 1k, Resistor_THT:R_Axial_DIN0207_L6.3mm_D2.5mm_P10.16mm_Horizontal, symbol Device:R
- removed R11, R12, R13, R6, R7, R8: 470, Resistor_THT:R_Axial_DIN0207_L6.3mm_D2.5mm_P10.16mm_Horizontal, symbol Device:R
- added RN1: 1k, Resistor_THT:R_Array_SIP7, symbol Device:R_Network06_Split
- added RN2: 470, Resistor_THT:R_Array_SIP7, symbol Device:R_Network06_Split
- added SW1: SW_DIP_x04, Package_DIP:DIP-8_W7.62mm, symbol Switch:SW_DIP_x04
- J2: footprint Connector_PinHeader_2.54mm:PinHeader_2x25_P2.54mm_Horizontal -> Connector_IDC:IDC-Header_2x25_P2.54mm_Horizontal
- J4: footprint Connector_Coaxial:BNC_Amphenol_B6252HB-NPP3G-50_Horizontal -> Z50-GDP:RCA_C160_Horizontal
- U1: footprint Package_DIP:DIP-40_W25.4mm -> Package_DIP:DIP-40_W15.24mm
- U9: value 74HCT273 -> 74LS273; symbol 74xx:74HCT273 -> 74xx:74LS273
- renumbered IC1 to U13
Connections:
- net +5V: now also RN1.1 (R1), RN1.1 (R1), RN1.1 (R1), RN1.1 (R1), RN1.1 (R1), RN1.1 (R1), RN2.1 (R1), RN2.1 (R1), RN2.1 (R1), RN2.1 (R1), RN2.1 (R1), RN2.1 (R1); no longer U1.21 (LPCK)
- net A2: now also U2.9; no longer U2.2
- net A3: now also U2.10; no longer U2.1
- net BAS: now also J5.5 (Pin_5); no longer J5.1 (Pin_1)
- net GND: now also J5.1 (Pin_1), SW1.1, SW1.2, SW1.3, SW1.4; no longer J5.5 (Pin_5)
- net HS: now also J3.10 (Pin_10), J3.12 (Pin_12), J5.4 (Pin_4); no longer J3.2 (Pin_2), J3.4 (Pin_4), J5.2 (Pin_2)
- net VI: now also J3.2 (Pin_2), J3.4 (Pin_4), J5.2 (Pin_2); no longer J3.10 (Pin_10), J3.12 (Pin_12), J5.4 (Pin_4)
- net ~{CAS}: now also U6.6; no longer U6.8
- net ~{INT}: now also RN1.6 (R5.2)
- net at U3.6: now also J3.3 (Pin_3), RN2.7 (R6.2); no longer J3.9 (Pin_9)
- net at U1.1 (CK), U10.12 (Cp), U7.12 (Q2)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: now also U6.4; no longer U6.10
- net at Q1.2 (B), R9.1: now also U3.4, RN2.6 (R5.2); no longer U3.10
- net at U12.13 (Qh), U3.5, U8.9: now also J3.1 (Pin_1); no longer J3.11 (Pin_11)
- net at U1.19 (~{MFREE}), U8.4: now also U6.9; no longer U6.2
- net at U2.6: now also U2.2; no longer U2.10
- net at U6.13: now also U2.3; no longer U2.8
- net at U4.6 (Oa=b), U5.3: now also U2.1; no longer U2.9
- net at U4.1 (B3): now also RN1.2 (R1.2), SW1.8
- net at U4.14 (B2): now also RN1.3 (R2.2), SW1.7
- net at U4.11 (B1): now also RN1.4 (R3.2), SW1.6
- net at U4.9 (B0): now also RN1.5 (R4.2), SW1.5
- net at U10.9 (Mr), U13.24 (OE): now also U6.3; no longer U6.6
- net at U2.4: now also U2.8; no longer U2.3
- net at J3.5 (Pin_5): now also U1.16 (VB), U3.11, RN2.4 (R3.2); no longer U3.4
- net at U1.22 (~{ALL}): now also U6.10; no longer U6.1
- net at U7.13 (Q1): now also U6.5; no longer U6.9
- new net: U1.34 (SYNC), U3.1, U3.3
- new net: J3.9 (Pin_9), RN2.2 (R1.2), U3.13, U3.2
- new net: J3.11 (Pin_11), RN2.3 (R2.2), U3.12
- new net: U10.2 (OE1), U10.3 (OE2), U6.1, U6.2, U6.8
- new net: J3.7 (Pin_7), RN2.5 (R4.2), U3.10
- new net: RN1.7 (R6.2), U1.21 (LPCK)

Commit message: Silkscreen
Parts:
- added JP1, JP2, JP3: SolderJumper_2_Bridged, Jumper:SolderJumper-2_P1.3mm_Bridged_RoundedPad1.0x1.5mm, symbol Jumper:SolderJumper_2_Bridged
Connections:
- net VI: now also JP1.1 (A), JP2.1 (A), JP3.1 (A)
- net at J6.3: now also JP3.2 (B)
- net at J6.4: now also JP2.2 (B)
- net at J6.5: now also JP1.2 (B)
- no-connect marks 43 -> 40
Other:
- moved on the sheet: J3, J4, J5, Q1, R10, R14, R15, R16, R9, RN1F, RN2A, RN2B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

Commit message: Schematic cleanup
Parts:
- Q1: value BC107 -> BC548; footprint Package_TO_SOT_THT:TO-18-3 -> Package_TO_SOT_THT:TO-92_Inline; symbol Transistor_BJT:BC107 -> Transistor_BJT:BC548
- RN1: value 1k -> 10k
Connections:
- net +5V: now also Q1.1 (C); no longer Q1.3 (C)
- net at R14.1, R16.1: now also Q1.3 (E); no longer Q1.1 (E)
- net 14M: no longer names the net of U12.7 (Clk), U7.2 (CP), U8.10, X1.5 (OUT)
Other:
- moved on the sheet: C1, C10, C11, C12, C13, C2, C3, C4, C5, C6, C7, C8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
